File: tmc2660-breakout.sch (KiCad schematic (older format))
At the start: 15 parts, among them P1 CONN_01X04, P2 CONN_01X02, P3 CONN_01X04, U1 TMC2660

Commit message: o little tweaks.
Parts:
- C4, C5: value CP -> 10u
- R2, R3: value R -> 10k
- R4, R5: value R -> 0.075
Other:
- moved on the sheet: C4, C5
Changed lines of the file:
@@
 L CP C4
 U 1 1 55767937
-P 4250 2100
-F 0 "C4" H 4275 2200 50  0000 L CNN
-F 1 "CP" H 4275 2000 50  0000 L CNN
-F 2 "Capacitors_SMD:C_1206" H 4288 1950 30  0001 C CNN
-F 3 "" H 4250 2100 60  0000 C CNN
-	1    4250 2100
-	0    -1   -1   0
+P 4800 2700
+F 0 "C4" H 4825 2800 50  0000 L CNN
+F 1 "10u" H 4825 2600 50  0000 L CNN
+F 2 "Capacitors_SMD:C_1206" H 4838 2550 30  0001 C CNN
+F 3 "" H 4800 2700 60  0000 C CNN
+	1    4800 2700
+	1    0    0    -1
 $EndComp
 $Comp
 L CP C5
 U 1 1 557679AB
-P 4250 2350
-F 0 "C5" H 4275 2450 50  0000 L CNN
-F 1 "CP" H 4275 2250 50  0000 L CNN
-F 2 "Capacitors_SMD:C_1206" H 4288 2200 30  0001 C CNN
-F 3 "" H 4250 2350 60  0000 C CNN
-	1    4250 2350
-	0    -1   -1   0
+P 4800 3550
+F 0 "C5" H 4825 3650 50  0000 L CNN
+F 1 "10u" H 4825 3450 50  0000 L CNN
+F 2 "Capacitors_SMD:C_1206" H 4838 3400 30  0001 C CNN
+F 3 "" H 4800 3550 60  0000 C CNN
+	1    4800 3550
+	1    0    0    -1
 $EndComp
 $Comp
 L GND #PWR01
 U 1 1 55767A6C
-P 4400 2100
-F 0 "#PWR01" H 4400 1850 50  0001 C CNN
-F 1 "GND" H 4400 1950 50  0000 C CNN
-F 2 "" H 4400 2100 60  0000 C CNN
-F 3 "" H 4400 2100 60  0000 C CNN
-	1    4400 2100
-	0    -1   -1   0
+P 4800 3700
+F 0 "#PWR01" H 4800 3450 50  0001 C CNN
+F 1 "GND" H 4800 3550 50  0000 C CNN
+F 2 "" H 4800 3700 60  0000 C CNN
+F 3 "" H 4800 3700 60  0000 C CNN
+	1    4800 3700
+	1    0    0    -1
 $EndComp
 $Comp
 L GND #PWR02
 U 1 1 55767A87
-P 4400 2350
-F 0 "#PWR02" H 4400 2100 50  0001 C CNN
-F 1 "GND" H 4400 2200 50  0000 C CNN
-F 2 "" H 4400 2350 60  0000 C CNN
-F 3 "" H 4400 2350 60  0000 C CNN
-	1    4400 2350
-	0    -1   -1   0
+P 4800 2850
+F 0 "#PWR02" H 4800 2600 50  0001 C CNN
+F 1 "GND" H 4800 2700 50  0000 C CNN
+F 2 "" H 4800 2850 60  0000 C CNN
+F 3 "" H 4800 2850 60  0000 C CNN
+	1    4800 2850
+	1    0    0    -1
 $EndComp
 $Comp
@@
 	3600 2000 3600 2400
 Wire Wire Line
-	4050 3400 3950 3400
-Wire Wire Line
-	4050 2050 4050 3400
-Wire Wire Line
-	4050 2350 4100 2350
-Connection ~ 4050 2550
-Wire Wire Line
-	3950 2550 4050 2550
-Wire Wire Line
-	4100 2100 4050 2100
-Connection ~ 4050 2350
+	3950 3400 4800 3400
+Wire Wire Line
+	3950 2550 4800 2550
 $Comp
 L C C3
@@
 P 4400 3250
 F 0 "R4" V 4480 3250 50  0000 C CNN
-F 1 "R" V 4400 3250 50  0000 C CNN
+F 1 "0.075" V 4400 3250 50  0000 C CNN
 F 2 "Resistors_SMD:R_1206" V 4330 3250 30  0001 C CNN
 F 3 "" H 4400 3250 30  0000 C CNN
@@
 P 4100 3150
 F 0 "R2" V 4180 3150 50  0000 C CNN
-F 1 "R" V 4100 3150 50  0000 C CNN
+F 1 "10k" V 4100 3150 50  0000 C CNN
 F 2 "Resistors_SMD:R_0805" V 4030 3150 30  0001 C CNN
 F 3 "" H 4100 3150 30  0000 C CNN
@@
 P 4100 4000
 F 0 "R3" V 4180 4000 50  0000 C CNN
-F 1 "R" V 4100 4000 50  0000 C CNN
+F 1 "10k" V 4100 4000 50  0000 C CNN
 F 2 "Resistors_SMD:R_0805" V 4030 4000 30  0001 C CNN
 F 3 "" H 4100 4000 30  0000 C CNN
@@
 P 4400 4100
 F 0 "R5" V 4480 4100 50  0000 C CNN
-F 1 "R" V 4400 4100 50  0000 C CNN
+F 1 "0.075" V 4400 4100 50  0000 C CNN
 F 2 "Resistors_SMD:R_1206" V 4330 4100 30  0001 C CNN
 F 3 "" H 4400 4100 30  0000 C CNN
@@
 	0    1    1    0
 $EndComp
-Text GLabel 4050 2050 1    60   Input ~ 0
+Text GLabel 4800 2500 1    60   Input ~ 0
 VMot
-Connection ~ 4050 2100
 $Comp
 L TMC2660 U1
@@
 	3950 2650 3950 2800
 Connection ~ 3950 2750
+Connection ~ 4050 3400
+Wire Wire Line
+	4800 2550 4800 2500
+Connection ~ 4800 2550
+Text GLabel 4800 3350 1    60   Input ~ 0
+VMot
+Wire Wire Line
+	4800 3400 4800 3350
+Connection ~ 4800 3400
 $EndSCHEMATC

Commit message: o First fully placed and routed.
Parts:
- added C6: 100n, Capacitors_SMD:C_0805, symbol C
- added P4: VCC, Pin_Headers:Pin_Header_Straight_1x02, symbol CONN_01X02
- added P5: VMOT, Pin_Headers:Pin_Header_Straight_1x02, symbol CONN_01X02
- C1: value C -> 470n
- C2, C3: value C -> 100n
- P1: value CONN_01X04 -> SPI
- P2: value CONN_01X02 -> StepDir
- P3: value CONN_01X04 -> Motor
Connections:
- net 1A1: now also P3.2 (P2); no longer P3.1 (P1)
- net 1A2: now also P3.1 (P1); no longer P3.2 (P2)
- net GND: now also U1.1 (NC), U1.19 (~EN), C6.2, P4.1 (P1), P5.1 (P1)
- net VMot: now also U1.33 (NC), P5.2 (P2)
- net at U1.40 (VCC): now also C6.1, P4.2 (P2)
- no-connect marks 0 -> 2
Other:
- moved on the sheet: P3
Changed lines of the file:
@@
 P 3450 2250
 F 0 "C2" H 3475 2350 50  0000 L CNN
-F 1 "C" H 3475 2150 50  0000 L CNN
+F 1 "100n" H 3250 2150 50  0000 L CNN
 F 2 "Capacitors_SMD:C_0805" H 3488 2100 30  0001 C CNN
 F 3 "" H 3450 2250 60  0000 C CNN
@@
 	1    0    0    -1
 $EndComp
-Text GLabel 3400 2000 0    60   Input ~ 0
+Text GLabel 2750 1950 1    60   Input ~ 0
 VMot
 Wire Wire Line
 	3450 2000 3450 2100
-Wire Wire Line
-	3400 2000 3750 2000
 Wire Wire Line
 	3600 2000 3600 2400
@@
 P 3750 2150
 F 0 "C3" H 3775 2250 50  0000 L CNN
-F 1 "C" H 3775 2050 50  0000 L CNN
+F 1 "100n" H 3775 2050 50  0000 L CNN
 F 2 "Capacitors_SMD:C_0805" H 3788 2000 30  0001 C CNN
 F 3 "" H 3750 2150 60  0000 C CNN
@@
 	0    -1   -1   0
 $EndComp
-$Comp
-L +3.3V #PWR07
-U 1 1 55768CBF
-P 2750 4000
-F 0 "#PWR07" H 2750 3850 50  0001 C CNN
-F 1 "+3.3V" H 2750 4140 50  0000 C CNN
-F 2 "" H 2750 4000 60  0000 C CNN
-F 3 "" H 2750 4000 60  0000 C CNN
-	1    2750 4000
-	0    -1   -1   0
-$EndComp
 Text GLabel 4150 2700 2    60   Output ~ 0
 1A1
@@
 L CONN_01X04 P3
 U 1 1 5576913F
-P 3450 1450
-F 0 "P3" H 3450 1700 50  0000 C CNN
-F 1 "CONN_01X04" V 3550 1450 50  0000 C CNN
-F 2 "Pin_Headers:Pin_Header_Straight_1x04" H 3450 1450 60  0001 C CNN
-F 3 "" H 3450 1450 60  0000 C CNN
-	1    3450 1450
-	0    -1   -1   0
-$EndComp
-Text GLabel 3300 1650 3    50   Input ~ 0
+P 5500 3400
+F 0 "P3" H 5500 3650 50  0000 C CNN
+F 1 "Motor" V 5600 3400 50  0000 C CNN
+F 2 "Pin_Headers:Pin_Header_Straight_1x04" H 5500 3400 60  0001 C CNN
+F 3 "" H 5500 3400 60  0000 C CNN
+	1    5500 3400
+	1    0    0    -1
+$EndComp
+Text GLabel 5300 3350 0    50   Input ~ 0
 1A1
-Text GLabel 3400 1650 3    50   Input ~ 0
+Text GLabel 5300 3250 0    50   Input ~ 0
 1A2
-Text GLabel 3500 1650 3    50   Input ~ 0
+Text GLabel 5300 3450 0    50   Input ~ 0
 1B1
-Text GLabel 3600 1650 3    50   Input ~ 0
+Text GLabel 5300 3550 0    50   Input ~ 0
 1B2
 $Comp
@@
 $EndComp
 $Comp
-L GND #PWR08
+L GND #PWR07
 U 1 1 55769BC1
 P 2200 3600
-F 0 "#PWR08" H 2200 3350 50  0001 C CNN
+F 0 "#PWR07" H 2200 3350 50  0001 C CNN
 F 1 "GND" H 2200 3450 50  0000 C CNN
 F 2 "" H 2200 3600 60  0000 C CNN
@@
 P 2350 3000
 F 0 "P1" H 2350 3250 50  0000 C CNN
-F 1 "CONN_01X04" V 2450 3000 50  0000 C CNN
+F 1 "SPI" V 2450 3000 50  0000 C CNN
 F 2 "Pin_Headers:Pin_Header_Straight_1x04" H 2350 3000 60  0001 C CNN
 F 3 "" H 2350 3000 60  0000 C CNN
@@
 P 2350 3350
 F 0 "P2" H 2350 3500 50  0000 C CNN
-F 1 "CONN_01X02" V 2450 3350 50  0000 C CNN
+F 1 "StepDir" V 2450 3350 50  0000 C CNN
 F 2 "Pin_Headers:Pin_Header_Straight_1x02" H 2350 3350 60  0001 C CNN
 F 3 "" H 2350 3350 60  0000 C CNN
@@
 P 2750 3850
 F 0 "C1" H 2775 3950 50  0000 L CNN
-F 1 "C" H 2775 3750 50  0000 L CNN
+F 1 "470n" V 2650 3600 50  0000 L CNN
 F 2 "Capacitors_SMD:C_0805" H 2788 3700 30  0001 C CNN
 F 3 "" H 2750 3850 60  0000 C CNN
@@
 $EndComp
 $Comp
-L GND #PWR09
+L GND #PWR08
 U 1 1 55769FFF
 P 2600 3850
-F 0 "#PWR09" H 2600 3600 50  0001 C CNN
+F 0 "#PWR08" H 2600 3600 50  0001 C CNN
 F 1 "GND" H 2600 3700 50  0000 C CNN
 F 2 "" H 2600 3850 60  0000 C CNN
@@
 $EndComp
 Wire Wire Line
-	2750 4000 2900 4000
-Wire Wire Line
 	4250 4000 4250 4100
 Wire Wire Line
@@
 	3950 2650 3950 2800
 Connection ~ 3950 2750
-Connection ~ 4050 3400
 Wire Wire Line
 	4800 2550 4800 2500
@@
 	4800 3400 4800 3350
 Connection ~ 4800 3400
+Text Label 4000 2700 0    60   ~ 0
+1A1
+Text Label 4000 3000 0    60   ~ 0
+1A2
+Text Label 4000 3600 0    60   ~ 0
+1B1
+Text Label 3950 3850 0    60   ~ 0
+1B2
+$Comp
+L CONN_01X02 P4
+U 1 1 5671135A
+P 2350 4050
+F 0 "P4" H 2350 4200 50  0000 C CNN
+F 1 "VCC" V 2450 4050 50  0000 C CNN
+F 2 "Pin_Headers:Pin_Header_Straight_1x02" H 2350 4050 60  0001 C CNN
+F 3 "" H 2350 4050 60  0000 C CNN
+	1    2350 4050
+	-1   0    0    1
+$EndComp
+$Comp
+L GND #PWR09
+U 1 1 56711446
+P 2650 4300
+F 0 "#PWR09" H 2650 4050 50  0001 C CNN
+F 1 "GND" H 2650 4150 50  0000 C CNN
+F 2 "" H 2650 4300 60  0000 C CNN
+F 3 "" H 2650 4300 60  0000 C CNN
+	1    2650 4300
+	1    0    0    -1
+$EndComp
+$Comp
+L C C6
+U 1 1 56711673
+P 2800 4150
+F 0 "C6" H 2825 4250 50  0000 L CNN
+F 1 "100n" H 2600 4050 50  0000 L CNN
+F 2 "Capacitors_SMD:C_0805" H 2838 4000 30  0001 C CNN
+F 3 "" H 2800 4150 60  0000 C CNN
+	1    2800 4150
+	1    0    0    -1
+$EndComp
+Connection ~ 2800 4000
+Wire Wire Line
+	2550 4100 2550 4300
+Wire Wire Line
+	2550 4300 2800 4300
+Connection ~ 2650 4300
+$Comp
+L CONN_01X02 P5
+U 1 1 5672E738
+P 2350 2050
+F 0 "P5" H 2350 2200 50  0000 C CNN
+F 1 "VMOT" V 2450 2050 50  0000 C CNN
+F 2 "Pin_Headers:Pin_Header_Straight_1x02" H 2350 2050 60  0001 C CNN
+F 3 "" H 2350 2050 60  0000 C CNN
+	1    2350 2050
+	-1   0    0    1
+$EndComp
+$Comp
+L GND #PWR010
+U 1 1 5672E81A
+P 2550 2150
+F 0 "#PWR010" H 2550 1900 50  0001 C CNN
+F 1 "GND" H 2550 2000 50  0000 C CNN
+F 2 "" H 2550 2150 60  0000 C CNN
+F 3 "" H 2550 2150 60  0000 C CNN
+	1    2550 2150
+	1    0    0    -1
+$EndComp
+Wire Wire Line
+	2550 2100 2550 2150
+Wire Wire Line
+	2550 2000 3750 2000
+Wire Wire Line
+	2750 1950 2750 2000
+Connection ~ 2750 2000
+NoConn ~ 2900 3700
+$Comp
+L GND #PWR011
+U 1 1 5672F758
+P 2650 2600
+F 0 "#PWR011" H 2650 2350 50  0001 C CNN
+F 1 "GND" H 2650 2450 50  0000 C CNN
+F 2 "" H 2650 2600 60  0000 C CNN
+F 3 "" H 2650 2600 60  0000 C CNN
+	1    2650 2600
+	1    0    0    -1
+$EndComp
+Wire Wire Line
+	2650 2600 2900 2600
+NoConn ~ 2900 2700
+Wire Wire Line
+	2900 3950 2850 3950
+Wire Wire Line
+	2850 4000 2850 3950
+Wire Wire Line
+	2550 4000 2850 4000
+Text GLabel 3150 4250 3    50   Input ~ 0
+VMot
+$Comp
+L GND #PWR?
+U 1 1 56739574
+P 3050 4250
+F 0 "#PWR?" H 3050 4000 50  0001 C CNN
+F 1 "GND" H 3000 4100 50  0000 C CNN
+F 2 "" H 3050 4250 60  0000 C CNN
+F 3 "" H 3050 4250 60  0000 C CNN
+	1    3050 4250
+	1    0    0    -1
+$EndComp
 $EndSCHEMATC
